Commit message: micky: WX200 setup of FBOT's micky robot
- urdf/wx200.urdf.xacro: ee_gripper TCP for micky's longer, offset gripper
  (0.020 0 0.02 instead of 0.027575 0 0)
- srdf/wx200.srdf.xacro: Grasping/Released gripper states for that gripper
  (left_finger 0.0195 / 0.030)
- xsarm_moveit.launch.py: load move_group/ExecuteTaskSolutionCapability
  (fbot_manipulator executes MoveIt Task Constructor solutions)
- interbotix_xsarm_control/config/wx200.yaml: motor 2/3 drive modes and
  gripper sleep position of micky's arm
- rviz/xsarm_moveit.rviz: RViz layout

The simulation (micky_description) keeps the stock gripper values.

Co-Authored-By: Claude Opus 5.5 <noreply@anthropic.com>

File: interbotix_ros_xsarms/interbotix_xsarm_descriptions/urdf/wx200.urdf.xacro (robot description, xacro)
@@ -633,5 +633,5 @@
           <origin
             rpy="0 0 0"
-            xyz="0.027575 0 0"/>
+            xyz="0.020 0 0.02"/>
           <parent
             link="$(arg robot_name)/fingers_link"/>

File: interbotix_ros_xsarms/interbotix_xsarm_moveit/config/srdf/wx200.srdf.xacro (robot description, xacro)
@@ -53,9 +53,9 @@
     </group_state>
     <group_state name="Grasping" group="interbotix_gripper">
-        <joint name="left_finger" value="0.015" />
+        <joint name="left_finger" value="0.0195" />
         <joint name="right_finger" value="-0.015" />
     </group_state>
     <group_state name="Released" group="interbotix_gripper">
-        <joint name="left_finger" value="0.037" />
+        <joint name="left_finger" value="0.030" />
         <joint name="right_finger" value="-0.037" />
     </group_state>
