Commit message: :eggplant: fix package

File: interbotix_ros_xsarms/interbotix_xsarm_descriptions/urdf/wx200.urdf.xacro (robot description, xacro)
@@ -633,5 +633,5 @@
           <origin
             rpy="0 0 0"
-            xyz="0.020 0 0.02"/>
+            xyz="0.020 0 0.02"/> <!--"0.027575 0 0"-->
           <parent
             link="$(arg robot_name)/fingers_link"/>

File: interbotix_ros_xsarms/interbotix_xsarm_moveit/config/srdf/wx200.srdf.xacro (robot description, xacro)
@@ -53,9 +53,9 @@
     </group_state>
     <group_state name="Grasping" group="interbotix_gripper">
-        <joint name="left_finger" value="0.0195" />
+        <joint name="left_finger" value="0.015" />
         <joint name="right_finger" value="-0.015" />
     </group_state>
     <group_state name="Released" group="interbotix_gripper">
-        <joint name="left_finger" value="0.030" />
+        <joint name="left_finger" value="0.037" />
         <joint name="right_finger" value="-0.037" />
     </group_state>
